File: _autosave-OLL.E fpv_pcb.kicad_sch (KiCad schematic)
At the start: 90 parts, among them J1 RC, J2 RC, J3 Conn_01x02_Pin, J4 M1 front left, J8 reciver, J9 TYPE-C-31-M-12, Q1 2N7002, U1 MP2315GJ, U13 BMP280, U14 STM32H753VITx, U15 USBLC6-2SC6, U2 W25Q128JVSIQ, U3 MP2315GJ, U4 ICM-42688-P, U5 UCC27511ADBV, U6 ul_AON7410, Y2 8HMz

Commit message: update desgin
Parts:
- removed J1: RC, Connector_PinHeader_2.54mm:PinHeader_1x04_P2.54mm_Vertical, symbol Connector:Conn_01x04_Pin
- added H1, H2, H3, H4: MountingHole, MountingHole:MountingHole_2.1mm, symbol Mechanical:MountingHole
- added J1: Micro_SD_Card, Connector_Card:microSD_HC_Wuerth_693072010801, symbol Connector:Micro_SD_Card
- added J10: Conn_01x05_Pin, Connector_PinHeader_1.00mm:PinHeader_1x05_P1.00mm_Vertical, symbol Connector:Conn_01x05_Pin
- C1, C10, C11, C12, C13, C14, C15, C16, C17, C18, C19, C2, C20, C21, C22, C23, C24, C25, C26, C3, C30, C32, C38, C39, C4, C40, C41, C42, C43, C44, C45, C46, C5, C6, C7, C8, C9: footprint Capacitor_SMD:C_0201_0603Metric_Pad0.64x0.40mm_HandSolder -> Capacitor_SMD:C_0603_1608Metric
- C1bulk1, C2bulk1: footprint Capacitor_SMD:C_0201_0603Metric_Pad0.64x0.40mm_HandSolder -> Capacitor_SMD:C_1206_3216Metric
- J2, J8: footprint Connector_PinHeader_2.54mm:PinHeader_1x04_P2.54mm_Vertical -> Connector_PinHeader_1.27mm:PinHeader_1x04_P1.27mm_Vertical
- J3, J4: footprint Connector_AMASS:AMASS_XT30UPB-M_1x02_P5.0mm_Vertical -> Connector_PinHeader_2.54mm:PinHeader_1x02_P2.54mm_Vertical
- JP1: footprint Jumper:Jumper_Harwin_S1621_P10.9mm -> Jumper:SolderJumper-2_P1.3mm_Open_RoundedPad1.0x1.5mm
- Y2: footprint Crystal:Crystal_SMD_3225-4Pin_3.2x2.5mm -> Crystal:Crystal_SMD_3215-2Pin_3.2x1.5mm
- renumbered ferritebead2 to fb2
Connections:
- net +3V3_FC: now also J10.2 (Pin_2)
- net +5V_FC: now also C22.2 (-), C44.1 (+), U1.2 (IN), U1.6 (EN/SYNC)
- net +VBAT: no longer C22.2 (-), C44.1 (+), U1.2 (IN), U1.6 (EN/SYNC)
- net GND: now also J10.5 (Pin_5)
- net SWCLK: now also J10.4 (Pin_4)
- net SWDIO: now also J10.3 (Pin_3)
- new net NRST: J10.1 (Pin_1)
Other:
- note added: "MP2315GJ"
- moved on the sheet: C13, R7, U2
