File: _autosave-OLL.E fpv_pcb.kicad_pcb (KiCad board)
At the start: 6 copper layers, 47.6 x 41.5 mm, 131 parts, among them J1 Micro_SD_Card, J10 Conn_01x05_Pin, J2 RC, J8 reciver, J9 TYPE-C-31-M-12, M1 M1 front left, M2 m4 rear left, M3 M2 front right, M4 M3 rear right, Q1 2N7002, SW1 SW_SPST, SW2 SW_SPST, U1 MP2315GJ, U10 AON7410, U11 UCC27511ADBV, U12 AON7410, U13 BMP280, U14 STM32H753VITx, U15 USBLC6-2SC6, U3 MP2315GJ, U4 ICM-42688-P, U5 UCC27511ADBV, U6 ul_AON7410, U7 UCC27511ADBV, U8 AON7410, U9 UCC27511ADBV, Y2 8HMz

Commit message: update pcb
Connections:
- D6 pad 1: +VBAT -> (no net)
Routing:
- net GND: track 141.0 -> 145.3 mm
Changed lines of the file:
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@@
 			(layers "F.Cu" "F.Mask" "F.Paste")
 			(roundrect_rratio 0.1388888889)
-			(net 3 "+VBAT")
 		)
 		(pad "2" smd roundrect
@@
 	)
 	(segment
+		(start 232.8 70.7)
+		(end 232.8 74.1)
+		(width 1)
+		(layer "F.Cu")
+		(net 1)
+	)
+	(segment
 		(start 212.7 59.3625)
 		(end 213.65 59.3625)
@@
 		(layer "F.Cu")
 		(net 1)
+	)
+	(segment
+		(start 232.8 74.1)
+		(end 233.4 74.7)
+		(width 1)
+		(layer "F.Cu")
+		(net 1)
