File: OLL.E fpv_pcb.kicad_sch (KiCad schematic)
At the start: 90 parts, among them J1 RC, J2 RC, J3 Conn_01x02_Pin, J4 M1 front left, J8 reciver, J9 TYPE-C-31-M-12, Q1 2N7002, U1 MP2315GJ, U13 BMP280, U14 STM32H753VITx, U15 USBLC6-2SC6, U2 W25Q128JVSIQ, U3 MP2315GJ, U4 ICM-42688-P, U5 UCC27511ADBV, U6 ul_AON7410, Y2 8HMz

Commit message: update desgin
Parts:
- removed J1: RC, Connector_PinHeader_2.54mm:PinHeader_1x04_P2.54mm_Vertical, symbol Connector:Conn_01x04_Pin
- added H1, H2, H3, H4: MountingHole, MountingHole:MountingHole_2.1mm, symbol Mechanical:MountingHole
- added J10: Conn_01x05_Pin, Connector_PinHeader_1.00mm:PinHeader_1x05_P1.00mm_Vertical, symbol Connector:Conn_01x05_Pin
- C1, C10, C11, C12, C13, C14, C15, C16, C17, C18, C19, C2, C20, C21, C22, C23, C24, C25, C26, C3, C30, C32, C38, C39, C4, C40, C41, C42, C43, C44, C5, C6, C7, C8, C9: footprint Capacitor_SMD:C_0201_0603Metric_Pad0.64x0.40mm_HandSolder -> Capacitor_SMD:C_0603_1608Metric
- C1bulk1, C2bulk1: footprint Capacitor_SMD:C_0201_0603Metric_Pad0.64x0.40mm_HandSolder -> Capacitor_SMD:C_1206_3216Metric
- C45: renamed from C1bulk2; footprint Capacitor_SMD:C_0201_0603Metric_Pad0.64x0.40mm_HandSolder -> Capacitor_SMD:C_0603_1608Metric
- C46: renamed from C1bulk3; footprint Capacitor_SMD:C_0201_0603Metric_Pad0.64x0.40mm_HandSolder -> Capacitor_SMD:C_0603_1608Metric
- J2, J8: footprint Connector_PinHeader_2.54mm:PinHeader_1x04_P2.54mm_Vertical -> Connector_PinHeader_1.27mm:PinHeader_1x04_P1.27mm_Vertical
- J3, J4: footprint Connector_AMASS:AMASS_XT30UPB-M_1x02_P5.0mm_Vertical -> Connector_PinHeader_2.54mm:PinHeader_1x02_P2.54mm_Vertical
- JP1: footprint Jumper:Jumper_Harwin_S1621_P10.9mm -> Jumper:SolderJumper-2_P1.3mm_Open_RoundedPad1.0x1.5mm
- Y2: footprint Crystal:Crystal_SMD_3225-4Pin_3.2x2.5mm -> Crystal:Crystal_SMD_3215-2Pin_3.2x1.5mm
- renumbered ferritebead2 to fb2
Connections:
- net +3V3_FC: now also J10.2 (Pin_2)
- net +5V_FC: now also C22.2 (-), C44.1 (+), U1.2 (IN), U1.6 (EN/SYNC)
- net +VBAT: now also D3.A; no longer C22.2 (-), C44.1 (+), D3.C, U1.2 (IN), U1.6 (EN/SYNC)
- net GND: now also J10.5 (Pin_5)
- net SWCLK: now also J10.4 (Pin_4)
- net SWDIO: now also J10.3 (Pin_3)
- net at C26.2 (-), J4.2 (Pin_2), U6.5 (D)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: now also D3.C; no longer D3.A
- new net NRST: J10.1 (Pin_1)
Other:
- note added: "MP2315GJ"
- moved on the sheet: D3

Commit message: update sd card
Parts:
- removed C13: 100nf, Capacitor_SMD:C_0603_1608Metric, symbol PCM_Elektuur:C
- removed R7: 10k, Resistor_SMD:R_0603_1608Metric, symbol PCM_Elektuur:R
- removed U2: W25Q128JVSIQ, Package_SO:SOIC-8-1EP_3.9x4.9mm_P1.27mm_EP2.29x3mm, symbol W25Q128JVSIQ:W25Q128JVSIQ
- added C47: 100nF, Capacitor_SMD:C_0603_1608Metric, symbol PCM_Elektuur:C
- added C48: 10uF, Capacitor_SMD:C_0603_1608Metric, symbol PCM_Elektuur:C
- added J1: Micro_SD_Card, Connector_Card:microSD_HC_Wuerth_693072010801, symbol Connector:Micro_SD_Card
- added R28, R29, R30, R31, R32: 47k, Resistor_SMD:R_0603_1608Metric, symbol PCM_Elektuur:R
Connections:
- net +3V3_FC: now also C47.1 (+), C48.1 (+), J1.4 (VDD), R28.1 (+), R29.1 (+), R30.1 (+), R31.2 (-), R32.1 (+)
- net +VBAT: now also D3.C; no longer D3.A
- net GND: now also C47.2 (-), C48.2 (-), J1.6 (VSS), J1.9 (SHIELD)
- net at C26.2 (-), J4.2 (Pin_2), U6.5 (D)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: now also D3.A; no longer D3.C
- net C1_D0: now reaches U14.65 (PC8)
- net C1_D0: now also J1.7 (DAT0), R29.2 (-)
- net C1_D1: now reaches U14.66 (PC9)
- net C1_D1: now also J1.8 (DAT1), R30.2 (-)
- net C1_D2: now reaches U14.78 (PC10)
- net C1_D2: now also J1.1 (DAT2), R28.2 (-)
- net C1_D3: now reaches U14.79 (PC11)
- net C1_D3: now also J1.2 (DAT3/CD), R32.2 (-)
- net CLK: now reaches U14.80 (PC12)
- net CLK: now also J1.5 (CLK)
- net CMD: now reaches U14.83 (PD2)
- net CMD: now also J1.3 (CMD), R31.1 (+)
- net CS_FLASH: no longer names the net of U14.51 (PB12)
- no-connect marks 56 -> 51
Other:
- note added: "SD CARD"
- note removed: "16MB = several minutes of 1kHz logging :gyro,motor outputs why its oscillated"
- note removed: "BLACKBOX FLASH"
- moved on the sheet: D3

Commit message: update IMU
Parts:
- removed JP1: Jumper_2_Open, Jumper:SolderJumper-2_P1.3mm_Open_RoundedPad1.0x1.5mm, symbol Jumper:Jumper_2_Open
- added SW1, SW2: SW_SPST, Button_Switch_SMD:SW_SPST_B3U-1000P, symbol Switch:SW_SPST
- J1: footprint Connector_Card:microSD_HC_Wuerth_693072010801 -> Connector_Card:microSD_HC_Hirose_DM3D-SF
Connections:
- net +3V3_FC: now also SW1.1 (A)
- net BOOT0: now also SW1.2 (B)
- net GND: now also SW2.2 (B)
- net at C41.1 (+), R21.1 (+), U14.14 (NRST): now also SW2.1 (A)
Changed lines of the file:
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@@
 	)
 	(junction
+		(at 394.97 27.94)
+		(diameter 0)
+		(color 0 0 0 0)
+	)
+	(junction
 		(at 288.29 20.32)
 		(diameter 0)
@@
 	)
 	(junction
-		(at 389.89 27.94)
-		(diameter 0)
-		(color 0 0 0 0)
-	)
-	(junction
 		(at 274.32 130.81)
 		(diameter 0)
@@
 	)
 	(junction
+		(at 316.23 39.37)
+		(diameter 0)
+		(color 0 0 0 0)
+	)
+	(junction
 		(at 290.83 204.47)
 		(diameter 0)
@@
 	(wire
 		(pts
-			(xy 389.89 27.94) (xy 397.51 27.94)
+			(xy 389.89 27.94) (xy 394.97 27.94)
 		)
 		(stroke
@@
 	(wire
 		(pts
+			(xy 316.23 39.37) (xy 316.23 46.99)
+		)
+		(stroke
+			(width 0)
+			(type default)
+		)
+	)
+	(wire
+		(pts
 			(xy 312.42 62.23) (xy 312.42 60.96)
 		)
@@
 	(wire
 		(pts
+			(xy 394.97 27.94) (xy 397.51 27.94)
+		)
+		(stroke
+			(width 0)
+			(type default)
+		)
+	)
+	(wire
+		(pts
 			(xy 370.84 59.69) (xy 382.27 59.69)
 		)
@@
 	(wire
 		(pts
+			(xy 386.08 25.4) (xy 394.97 25.4)
+		)
+		(stroke
+			(width 0)
+			(type default)
+		)
+	)
+	(wire
+		(pts
 			(xy 278.13 57.15) (xy 274.32 57.15)
 		)
@@
 	(wire
 		(pts
-			(xy 316.23 36.83) (xy 316.23 46.99)
+			(xy 316.23 36.83) (xy 316.23 39.37)
 		)
 		(stroke
@@
 	(wire
 		(pts
+			(xy 383.54 27.94) (xy 386.08 27.94)
+		)
+		(stroke
+			(width 0)
+			(type default)
+		)
+	)
+	(wire
+		(pts
 			(xy 266.7 267.97) (xy 270.51 267.97)
 		)
@@
 	(wire
 		(pts
+			(xy 386.08 27.94) (xy 386.08 25.4)
+		)
+		(stroke
+			(width 0)
+			(type default)
+		)
+	)
+	(wire
+		(pts
 			(xy 283.21 250.19) (xy 283.21 251.46)
 		)
@@
 	(wire
 		(pts
-			(xy 383.54 27.94) (xy 389.89 27.94)
-		)
-		(stroke
-			(width 0)
-			(type default)
-		)
-	)
-	(wire
-		(pts
 			(xy 295.91 260.35) (xy 294.64 260.35)
 		)
@@
 	(wire
 		(pts
+			(xy 394.97 25.4) (xy 394.97 27.94)
+		)
+		(stroke
+			(width 0)
+			(type default)
+		)
+	)
+	(wire
+		(pts
 			(xy 267.97 30.48) (xy 274.32 30.48)
 		)
@@
 	)
 	(symbol
-		(lib_id "Jumper:Jumper_2_Open")
-		(at 378.46 27.94 0)
-		(unit 1)
-		(exclude_from_sim no)
-		(in_bom yes)
-		(on_board yes)
-		(dnp no)
-		(fields_autoplaced yes)
-		(property "Reference" "JP1"
-			(at 378.46 21.59 0)
-			(effects
-				(font
-					(size 1.27 1.27)
-				)
-			)
-		)
-		(property "Value" "Jumper_2_Open"
-			(at 378.46 24.13 0)
-			(effects
-				(font
-					(size 1.27 1.27)
-				)
-			)
-		)
-		(property "Footprint" "Jumper:SolderJumper-2_P1.3mm_Open_RoundedPad1.0x1.5mm"
-			(at 378.46 27.94 0)
-			(effects
-				(font
-					(size 1.27 1.27)
-				)
-				(hide yes)
-			)
-		)
-		(property "Datasheet" "~"
-			(at 378.46 27.94 0)
-			(effects
-				(font
-					(size 1.27 1.27)
-				)
-				(hide yes)
-			)
-		)
-		(property "Description" "Jumper, 2-pole, open"
-			(at 378.46 27.94 0)
-			(effects
-				(font
-					(size 1.27 1.27)
-				)
-				(hide yes)
-			)
-		)
-		(pin "1"
-		)
-		(pin "2"
-		)
-		(instances
-			(project "OLL.E fpv_pcb"
-				(path "/7062ecae-ed82-47dc-bd4a-f40d8cc668c3"
-					(reference "JP1")
-					(unit 1)
-				)
-			)
-		)
-	)
-	(symbol
 		(lib_id "power:GND")
 		(at 58.42 121.92 0)
@@
 	(symbol
 		(lib_id "power:GND")
+		(at 326.39 39.37 0)
+		(unit 1)
+		(exclude_from_sim no)
+		(in_bom yes)
+		(on_board yes)
+		(dnp no)
+		(fields_autoplaced yes)
+		(property "Reference" "#PWR016"
+			(at 326.39 45.72 0)
+			(effects
+				(font
+					(size 1.27 1.27)
+				)
+				(hide yes)
+			)
+		)
+		(property "Value" "GND"
+			(at 326.39 44.45 0)
+			(effects
+				(font
+					(size 1.27 1.27)
+				)
+			)
+		)
+		(property "Footprint" ""
+			(at 326.39 39.37 0)
+			(effects
+				(font
+					(size 1.27 1.27)
+				)
+				(hide yes)
+			)
+		)
+		(property "Datasheet" ""
+			(at 326.39 39.37 0)
+			(effects
+				(font
+					(size 1.27 1.27)
+				)
+				(hide yes)
+			)
+		)
+		(property "Description" "Power symbol creates a global label with name \"GND\" , ground"
+			(at 326.39 39.37 0)
+			(effects
+				(font
+					(size 1.27 1.27)
+				)
+				(hide yes)
+			)
+		)
+		(pin "1"
+		)
+		(instances
+			(project "OLL.E fpv_pcb"
+				(path "/7062ecae-ed82-47dc-bd4a-f40d8cc668c3"
+					(reference "#PWR016")
+					(unit 1)
+				)
+			)
+		)
+	)
+	(symbol
+		(lib_id "power:GND")
 		(at 257.81 160.02 0)
 		(unit 1)
@@
 	)
 	(symbol
+		(lib_id "Switch:SW_SPST")
+		(at 321.31 39.37 0)
+		(unit 1)
+		(exclude_from_sim no)
+		(in_bom yes)
+		(on_board yes)
+		(dnp no)
+		(fields_autoplaced yes)
+		(property "Reference" "SW2"
+			(at 321.31 33.02 0)
+			(effects
+				(font
+					(size 1.27 1.27)
+				)
+			)
+		)
+		(property "Value" "SW_SPST"
+			(at 321.31 35.56 0)
+			(effects
+				(font
+					(size 1.27 1.27)
+				)
+			)
+		)
+		(property "Footprint" "Button_Switch_SMD:SW_SPST_B3U-1000P"
+			(at 321.31 39.37 0)
+			(effects
+				(font
+					(size 1.27 1.27)
+				)
+				(hide yes)
+			)
+		)
+		(property "Datasheet" "~"
+			(at 321.31 39.37 0)
+			(effects
+				(font
+					(size 1.27 1.27)
+				)
+				(hide yes)
+			)
+		)
+		(property "Description" "Single Pole Single Throw (SPST) switch"
+			(at 321.31 39.37 0)
+			(effects
+				(font
+					(size 1.27 1.27)
+				)
+				(hide yes)
+			)
+		)
+		(pin "1"
+		)
+		(pin "2"
+		)
+		(instances
+			(project "OLL.E fpv_pcb"
+				(path "/7062ecae-ed82-47dc-bd4a-f40d8cc668c3"
+					(reference "SW2")
+					(unit 1)
+				)
+			)
+		)
+	)
+	(symbol
 		(lib_id "Diode:1N4148W")
 		(at 171.45 118.11 270)
@@
 	)
 	(symbol
+		(lib_id "Switch:SW_SPST")
+		(at 378.46 27.94 0)
+		(unit 1)
+		(exclude_from_sim no)
+		(in_bom yes)
+		(on_board yes)
+		(dnp no)
+		(fields_autoplaced yes)
+		(property "Reference" "SW1"
+			(at 378.46 21.59 0)
+			(effects
+				(font
+					(size 1.27 1.27)
+				)
+			)
+		)
+		(property "Value" "SW_SPST"
+			(at 378.46 24.13 0)
+			(effects
+				(font
+					(size 1.27 1.27)
+				)
+			)
+		)
+		(property "Footprint" "Button_Switch_SMD:SW_SPST_B3U-1000P"
+			(at 378.46 27.94 0)
+			(effects
+				(font
+					(size 1.27 1.27)
+				)
+				(hide yes)
+			)
+		)
+		(property "Datasheet" "~"
+			(at 378.46 27.94 0)
+			(effects
+				(font
+					(size 1.27 1.27)
+				)
+				(hide yes)
+			)
+		)
+		(property "Description" "Single Pole Single Throw (SPST) switch"
+			(at 378.46 27.94 0)
+			(effects
+				(font
+					(size 1.27 1.27)
+				)
+				(hide yes)
+			)
+		)
+		(pin "1"
+		)
+		(pin "2"
+		)
+		(instances
+			(project "OLL.E fpv_pcb"
+				(path "/7062ecae-ed82-47dc-bd4a-f40d8cc668c3"
+					(reference "SW1")
+					(unit 1)
+				)
+			)
+		)
+	)
+	(symbol
 		(lib_id "Device:Crystal")
 		(at 308.61 64.77 0)
@@
 			)
 		)
-		(property "Footprint" "Connector_Card:microSD_HC_Wuerth_693072010801"
+		(property "Footprint" "Connector_Card:microSD_HC_Hirose_DM3D-SF"
 			(at 7.62 48.26 0)
 			(effects

Commit message: update UART track 0.2mm
Parts:
- renumbered J3 to BAT1, J4 to M1
Connections:
- net +VBAT: now also D3.A; no longer D3.C
- net at C26.2 (-), M1.2 (Pin_2), U6.5 (D)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: now also D3.C; no longer D3.A
Other:
- moved on the sheet: D3
Changed lines of the file:
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@@
 	)
 	(junction
-		(at 170.18 176.53)
-		(diameter 0)
-		(color 0 0 0 0)
-	)
-	(junction
 		(at 266.7 147.32)
 		(diameter 0)
@@
 	)
 	(junction
+		(at 181.61 165.1)
+		(diameter 0)
+		(color 0 0 0 0)
+	)
+	(junction
 		(at 119.38 93.98)
 		(diameter 0)
@@
 	)
 	(junction
+		(at 170.18 176.53)
+		(diameter 0)
+		(color 0 0 0 0)
+	)
+	(junction
+		(at 161.29 176.53)
+		(diameter 0)
+		(color 0 0 0 0)
+	)
+	(junction
 		(at 31.75 88.9)
 		(diameter 0)
@@
 	)
 	(junction
+		(at 170.18 166.37)
+		(diameter 0)
+		(color 0 0 0 0)
+	)
+	(junction
 		(at 59.69 261.62)
 		(diameter 0)
@@
 	)
 	(junction
-		(at 161.29 176.53)
-		(diameter 0)
-		(color 0 0 0 0)
-	)
-	(junction
 		(at 257.81 151.13)
 		(diameter 0)
@@
 		(color 0 0 0 0)
 	)
-	(junction
-		(at 181.61 166.37)
-		(diameter 0)
-		(color 0 0 0 0)
-	)
-	(junction
-		(at 170.18 166.37)
-		(diameter 0)
-		(color 0 0 0 0)
-	)
 	(no_connect
 		(at 370.84 168.91)
@@
 	(wire
 		(pts
-			(xy 181.61 158.75) (xy 181.61 166.37)
+			(xy 181.61 158.75) (xy 181.61 165.1)
 		)
 		(stroke
@@
 	(wire
 		(pts
-			(xy 170.18 166.37) (xy 181.61 166.37)
-		)
-		(stroke
-			(width 0)
-			(type default)
-		)
-	)
-	(wire
-		(pts
 			(xy 62.23 20.32) (xy 64.77 20.32)
 		)
@@
 	(wire
 		(pts
-			(xy 161.29 176.53) (xy 170.18 176.53)
-		)
-		(stroke
-			(width 0)
-			(type default)
-		)
-	)
-	(wire
-		(pts
 			(xy 86.36 88.9) (xy 86.36 93.98)
 		)
@@
 	(wire
 		(pts
-			(xy 170.18 176.53) (xy 181.61 176.53)
-		)
-		(stroke
-			(width 0)
-			(type default)
-		)
-	)
-	(wire
-		(pts
 			(xy 53.34 162.56) (xy 59.69 162.56)
 		)
@@
 	(wire
 		(pts
-			(xy 160.02 166.37) (xy 170.18 166.37)
+			(xy 180.34 165.1) (xy 181.61 165.1)
 		)
 		(stroke
@@
 	(wire
 		(pts
+			(xy 181.61 165.1) (xy 181.61 166.37)
+		)
+		(stroke
+			(width 0)
+			(type default)
+		)
+	)
+	(wire
+		(pts
 			(xy 383.54 27.94) (xy 386.08 27.94)
 		)
@@
 	(wire
 		(pts
+			(xy 161.29 176.53) (xy 170.18 176.53)
+		)
+		(stroke
+			(width 0)
+			(type default)
+		)
+	)
+	(wire
+		(pts
 			(xy 313.69 26.67) (xy 321.31 26.67)
 		)
@@
 	(wire
 		(pts
+			(xy 170.18 166.37) (xy 180.34 166.37)
+		)
+		(stroke
+			(width 0)
+			(type default)
+		)
+	)
+	(wire
+		(pts
 			(xy 152.4 118.11) (xy 152.4 120.65)
 		)
@@
 	(wire
 		(pts
+			(xy 170.18 176.53) (xy 181.61 176.53)
+		)
+		(stroke
+			(width 0)
+			(type default)
+		)
+	)
+	(wire
+		(pts
 			(xy 67.31 40.64) (xy 68.58 40.64)
 		)
@@
 	(wire
 		(pts
+			(xy 160.02 166.37) (xy 170.18 166.37)
+		)
+		(stroke
+			(width 0)
+			(type default)
+		)
+	)
+	(wire
+		(pts
 			(xy 59.69 186.69) (xy 59.69 189.23)
 		)
@@
 	(wire
 		(pts
+			(xy 180.34 166.37) (xy 180.34 165.1)
+		)
+		(stroke
+			(width 0)
+			(type default)
+		)
+	)
+	(wire
+		(pts
 			(xy 280.67 255.27) (xy 283.21 255.27)
 		)
@@
 		(dnp no)
 		(fields_autoplaced yes)
-		(property "Reference" "J4"
+		(property "Reference" "M1"
 			(at 155.575 161.29 0)
 			(effects
@@
 			(project "OLL.E fpv_pcb"
 				(path "/7062ecae-ed82-47dc-bd4a-f40d8cc668c3"
-					(reference "J4")
+					(reference "M1")
 					(unit 1)
 				)
@@
 	(symbol
 		(lib_id "SS54FSH:SS54FSH")
-		(at 170.18 171.45 90)
+		(at 170.18 171.45 270)
 		(unit 1)
 		(exclude_from_sim no)
@@
 					(size 1.27 1.27)
 				)
-				(justify right)
+				(justify left)
 			)
 		)
@@
 					(size 1.27 1.27)
 				)
-				(justify right)
+				(justify left)
 			)
 		)
@@
 		(dnp no)
 		(fields_autoplaced yes)
-		(property "Reference" "J3"
+		(property "Reference" "BAT1"
 			(at 211.455 82.55 0)
 			(effects
@@
 			(project "OLL.E fpv_pcb"
 				(path "/7062ecae-ed82-47dc-bd4a-f40d8cc668c3"
-					(reference "J3")
+					(reference "BAT1")
 					(unit 1)
 				)

Commit message: latest update review the board
Connections:
- net +5V_FC: now also D7.2 (A); no longer D7.1 (K)
- net NRST: now also C41.1 (+), R21.1 (+), SW2.1 (A), U14.14 (NRST)
- net at LS1.N, Q1.3 (D): now also D7.1 (K); no longer D7.2 (A)
Other:
- moved on the sheet: D7
Changed lines of the file:
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@@
 		)
 	)
+	(global_label "NRST"
+		(shape bidirectional)
+		(at 316.23 46.99 180)
+		(fields_autoplaced yes)
+		(effects
+			(font
+				(size 1.27 1.27)
+			)
+			(justify right)
+		)
+		(property "Intersheetrefs" "${INTERSHEET_REFS}"
+			(at 307.3559 46.99 0)
+			(effects
+				(font
+					(size 1.27 1.27)
+				)
+				(justify right)
+				(hide yes)
+			)
+		)
+	)
 	(global_label "+3V3_FC"
 		(shape input)
@@
 	(symbol
 		(lib_id "Diode:1N4148W")
-		(at 171.45 118.11 270)
+		(at 171.45 118.11 90)
 		(unit 1)
 		(exclude_from_sim no)
@@
 		(dnp no)
 		(property "Reference" "D7"
-			(at 165.1 115.824 90)
+			(at 177.8 120.396 90)
 			(effects
 				(font
@@
 		)
 		(property "Value" "1N4148W"
-			(at 159.766 119.126 90)
+			(at 183.134 117.094 90)
 			(effects
 				(font
@@
 		)
 		(property "Footprint" "Diode_SMD:D_SOD-123"
-			(at 167.005 118.11 0)
+			(at 175.895 118.11 0)
 			(effects
 				(font
