File: untitled.kicad_sch (KiCad schematic)
At the start: 27 parts, among them J5 M2 front right, J6 M3 rear right, J7 m4 rear left, U10 AON7410, U11 UCC27511ADBV, U12 AON7410, U7 UCC27511ADBV, U8 AON7410, U9 UCC27511ADBV

Commit message: update desgin
Parts:
- C27, C28, C29, C31, C33, C34, C35, C36, C37: footprint Capacitor_SMD:C_0201_0603Metric_Pad0.64x0.40mm_HandSolder -> Capacitor_SMD:C_0603_1608Metric
- J5, J6, J7: footprint Connector_AMASS:AMASS_XT30UPB-M_1x02_P5.0mm_Vertical -> Connector_PinHeader_2.54mm:PinHeader_1x02_P2.54mm_Vertical
Changed lines of the file:
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@@
 	)
 	(junction
-		(at 162.56 41.91)
-		(diameter 0)
-		(color 0 0 0 0)
-	)
-	(junction
 		(at 139.7 44.45)
 		(diameter 0)
@@
 	)
 	(junction
-		(at 152.4 41.91)
-		(diameter 0)
-		(color 0 0 0 0)
-	)
-	(junction
 		(at 96.52 41.91)
 		(diameter 0)
@@
 	)
 	(junction
-		(at 162.56 31.75)
-		(diameter 0)
-		(color 0 0 0 0)
-	)
-	(junction
 		(at 160.02 144.78)
 		(diameter 0)
@@
 	)
 	(junction
+		(at 162.56 41.91)
+		(diameter 0)
+		(color 0 0 0 0)
+	)
+	(junction
 		(at 156.21 104.14)
 		(diameter 0)
@@
 	)
 	(junction
+		(at 173.99 31.75)
+		(diameter 0)
+		(color 0 0 0 0)
+	)
+	(junction
 		(at 54.61 130.81)
 		(diameter 0)
@@
 	)
 	(junction
+		(at 162.56 31.75)
+		(diameter 0)
+		(color 0 0 0 0)
+	)
+	(junction
 		(at 59.69 154.94)
 		(diameter 0)
@@
 	)
 	(junction
+		(at 152.4 41.91)
+		(diameter 0)
+		(color 0 0 0 0)
+	)
+	(junction
 		(at 95.25 146.05)
 		(diameter 0)
@@
 	)
 	(junction
-		(at 173.99 31.75)
-		(diameter 0)
-		(color 0 0 0 0)
-	)
-	(junction
 		(at 59.69 130.81)
 		(diameter 0)
@@
 	(wire
 		(pts
-			(xy 162.56 31.75) (xy 173.99 31.75)
-		)
-		(stroke
-			(width 0)
-			(type default)
-		)
-	)
-	(wire
-		(pts
 			(xy 208.28 104.14) (xy 208.28 106.68)
 		)
@@
 	(wire
 		(pts
+			(xy 152.4 41.91) (xy 162.56 41.91)
+		)
+		(stroke
+			(width 0)
+			(type default)
+		)
+	)
+	(wire
+		(pts
 			(xy 173.99 24.13) (xy 173.99 31.75)
 		)
@@
 	(wire
 		(pts
-			(xy 130.81 97.79) (xy 146.05 97.79)
+			(xy 162.56 41.91) (xy 173.99 41.91)
 		)
 		(stroke
@@
 	(wire
 		(pts
-			(xy 36.83 38.1) (xy 41.91 38.1)
+			(xy 130.81 97.79) (xy 146.05 97.79)
 		)
 		(stroke
@@
 	(wire
 		(pts
-			(xy 177.8 24.13) (xy 173.99 24.13)
+			(xy 36.83 38.1) (xy 41.91 38.1)
 		)
 		(stroke
@@
 	(wire
 		(pts
-			(xy 170.18 134.62) (xy 181.61 134.62)
+			(xy 177.8 24.13) (xy 173.99 24.13)
 		)
 		(stroke
@@
 	(wire
 		(pts
-			(xy 69.85 146.05) (xy 95.25 146.05)
+			(xy 170.18 134.62) (xy 181.61 134.62)
 		)
 		(stroke
@@
 	(wire
 		(pts
-			(xy 147.32 142.24) (xy 147.32 144.78)
+			(xy 69.85 146.05) (xy 95.25 146.05)
 		)
 		(stroke
@@
 	(wire
 		(pts
-			(xy 231.14 101.6) (xy 242.57 101.6)
+			(xy 147.32 142.24) (xy 147.32 144.78)
 		)
 		(stroke
@@
 	(wire
 		(pts
-			(xy 152.4 41.91) (xy 162.56 41.91)
+			(xy 231.14 101.6) (xy 242.57 101.6)
 		)
 		(stroke
@@
 	(wire
 		(pts
-			(xy 152.4 31.75) (xy 162.56 31.75)
+			(xy 205.74 106.68) (xy 208.28 106.68)
 		)
 		(stroke
@@
 	(wire
 		(pts
-			(xy 205.74 106.68) (xy 208.28 106.68)
+			(xy 69.85 140.97) (xy 85.09 140.97)
 		)
 		(stroke
@@
 	(wire
 		(pts
-			(xy 69.85 140.97) (xy 85.09 140.97)
+			(xy 59.69 130.81) (xy 59.69 135.89)
 		)
 		(stroke
@@
 	(wire
 		(pts
-			(xy 59.69 130.81) (xy 59.69 135.89)
+			(xy 170.18 144.78) (xy 181.61 144.78)
 		)
 		(stroke
@@
 	(wire
 		(pts
-			(xy 170.18 144.78) (xy 181.61 144.78)
+			(xy 165.1 106.68) (xy 161.29 106.68)
 		)
 		(stroke
@@
 	(wire
 		(pts
-			(xy 165.1 106.68) (xy 161.29 106.68)
+			(xy 205.74 99.06) (xy 208.28 99.06)
 		)
 		(stroke
@@
 	(wire
 		(pts
-			(xy 205.74 99.06) (xy 208.28 99.06)
+			(xy 152.4 31.75) (xy 162.56 31.75)
 		)
 		(stroke
@@
 	(wire
 		(pts
-			(xy 162.56 41.91) (xy 173.99 41.91)
+			(xy 99.06 144.78) (xy 104.14 144.78)
 		)
 		(stroke
@@
 	(wire
 		(pts
-			(xy 99.06 144.78) (xy 104.14 144.78)
+			(xy 46.99 154.94) (xy 59.69 154.94)
 		)
 		(stroke
@@
 	(wire
 		(pts
-			(xy 46.99 154.94) (xy 59.69 154.94)
+			(xy 44.45 140.97) (xy 49.53 140.97)
 		)
 		(stroke
@@
 	(wire
 		(pts
-			(xy 44.45 140.97) (xy 49.53 140.97)
+			(xy 162.56 31.75) (xy 173.99 31.75)
 		)
 		(stroke
@@
 			)
 		)
-		(property "Footprint" "Capacitor_SMD:C_0201_0603Metric_Pad0.64x0.40mm_HandSolder"
+		(property "Footprint" "Capacitor_SMD:C_0603_1608Metric"
 			(at 54.61 125.73 0)
 			(effects
@@
 			)
 		)
-		(property "Footprint" "Capacitor_SMD:C_0201_0603Metric_Pad0.64x0.40mm_HandSolder"
+		(property "Footprint" "Capacitor_SMD:C_0603_1608Metric"
 			(at 181.61 139.7 0)
 			(effects
@@
 			)
 		)
-		(property "Footprint" "Capacitor_SMD:C_0201_0603Metric_Pad0.64x0.40mm_HandSolder"
+		(property "Footprint" "Capacitor_SMD:C_0603_1608Metric"
 			(at 173.99 36.83 0)
 			(effects
@@
 			)
 		)
-		(property "Footprint" "Capacitor_SMD:C_0201_0603Metric_Pad0.64x0.40mm_HandSolder"
+		(property "Footprint" "Capacitor_SMD:C_0603_1608Metric"
 			(at 115.57 82.55 0)
 			(effects
@@
 			)
 		)
-		(property "Footprint" "Capacitor_SMD:C_0201_0603Metric_Pad0.64x0.40mm_HandSolder"
+		(property "Footprint" "Capacitor_SMD:C_0603_1608Metric"
 			(at 57.15 27.94 0)
 			(effects
@@
 			)
 		)
-		(property "Footprint" "Capacitor_SMD:C_0201_0603Metric_Pad0.64x0.40mm_HandSolder"
+		(property "Footprint" "Capacitor_SMD:C_0603_1608Metric"
 			(at 46.99 22.86 0)
 			(effects
@@
 			)
 		)
-		(property "Footprint" "Connector_AMASS:AMASS_XT30UPB-M_1x02_P5.0mm_Vertical"
+		(property "Footprint" "Connector_PinHeader_2.54mm:PinHeader_1x02_P2.54mm_Vertical"
 			(at 215.9 91.44 0)
 			(effects
@@
 			)
 		)
-		(property "Footprint" "Connector_AMASS:AMASS_XT30UPB-M_1x02_P5.0mm_Vertical"
+		(property "Footprint" "Connector_PinHeader_2.54mm:PinHeader_1x02_P2.54mm_Vertical"
 			(at 147.32 31.75 0)
 			(effects
@@
 			)
 		)
-		(property "Footprint" "Capacitor_SMD:C_0201_0603Metric_Pad0.64x0.40mm_HandSolder"
+		(property "Footprint" "Capacitor_SMD:C_0603_1608Metric"
 			(at 64.77 130.81 0)
 			(effects
@@
 			)
 		)
-		(property "Footprint" "Connector_AMASS:AMASS_XT30UPB-M_1x02_P5.0mm_Vertical"
+		(property "Footprint" "Connector_PinHeader_2.54mm:PinHeader_1x02_P2.54mm_Vertical"
 			(at 154.94 134.62 0)
 			(effects
@@
 			)
 		)
-		(property "Footprint" "Capacitor_SMD:C_0201_0603Metric_Pad0.64x0.40mm_HandSolder"
+		(property "Footprint" "Capacitor_SMD:C_0603_1608Metric"
 			(at 125.73 87.63 0)
 			(effects
@@
 			)
 		)
-		(property "Footprint" "Capacitor_SMD:C_0201_0603Metric_Pad0.64x0.40mm_HandSolder"
+		(property "Footprint" "Capacitor_SMD:C_0603_1608Metric"
 			(at 242.57 96.52 0)
 			(effects

Commit message: update UART track 0.2mm
Parts:
- renumbered J5 to M2, J6 to M3, J7 to M4
Connections:
- net +VBAT: now also D4.A, D5.A, D6.A; no longer D4.C, D5.C, D6.C
- net at C27.2 (-), M2.2 (Pin_2), U8.5 (D)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: now also D4.C; no longer D4.A
- net at C29.2 (-), M4.2 (Pin_2), U12.5 (D)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: now also D6.C; no longer D6.A
- net at C28.2 (-), M3.2 (Pin_2), U10.5 (D)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: now also D5.C; no longer D5.A
Other:
- moved on the sheet: D4, D5, D6

Commit message: update
Other:
- moved on the sheet: C28, C34, C35, D5, M3, R15, R16, U10, U9

Commit message: update scemetic desgin deleted bulk capictor fix all blocker
Parts:
- added C44, C49, C50: 22uF, Capacitor_SMD:C_1210_3225Metric, symbol PCM_Elektuur:C
Connections:
- net +VBAT: now also C44.2 (-), C49.2 (-), C50.2 (-)
- net GND: now also C44.1 (+), C49.1 (+), C50.1 (+)
